File: pcb/rcs-controller-sch-power.kicad_sch (KiCad schematic)
At the start: 63 parts, among them J1 00222-32051, J10 0022-232021, J2 0022-232021, J3 0022-232041, J8 00222-32051, Q1 SI7465DP-T1-E3, U2 MP26123DR-LF-Z, U3 TPS63070

Commit message: Finished BOM, changed holes to .3
Parts:
- renumbered C26 to C1, C11 to C10, C13 to C11, C14 to C12, C15 to C13, C16 to C14, C29 to C15, C1 to C2, C2 to C3, C6 to C5, C7 to C6, C8 to C7, C9 to C8, C10 to C9, D13 to D1, D1 to D2, D2 to D3, D9 to D4, D4 to D5, D5 to D6, J10 to J1, J8 to J2, J1 to J3, J2 to J4, J3 to J5, R35 to R1, R36 to R2, R1 to R3, R2 to R4, R3 to R5, R4 to R6, R5 to R7, R6 to R8, TP7 to TP10, TP9 to TP11, TP32 to TP6, TP30 to TP7, TP31 to TP8, TP6 to TP9, U2 to U1, U3 to U2
