File: pcb/rcs-controller-sch-microcontroller.kicad_sch (KiCad schematic)
At the start: 42 parts, among them J11 Conn_01x03, J4 Screw_Terminal_4_P3.50mm, J5 USB_C_Receptacle_USB2.0_14P, J6 Conn_01x03, J9 Conn_01x03, Q2 SI7465DP-T1-E3, Q3 SI7465DP-T1-E3, Q4 PMV45EN2, Q5 PMV45EN2, SW1 SW_Push, SW2 SW_Push, U1 LSM6DSOX, U4 ESP32-S3-WROOM-1

Commit message: Finished BOM, changed holes to .3
Parts:
- D8: DPN (none) -> 732-4979-1-ND; DST (none) -> DigiKey; MFR (none) -> Wurth; MPN (none) -> 150060SS75000
- J10: renamed from J11; value Conn_01x03 -> 0022232031; DPN (none) -> WM4201-ND; DST (none) -> DigiKey; MFR (none) -> Molex; MPN (none) -> 22232031
- J7: renamed from J6; value Conn_01x03 -> 0022232031; footprint Connector_PinHeader_2.54mm:PinHeader_1x03_P2.54mm_Vertical -> Connector_Molex:Molex_KK-254_AE-6410-03A_1x03_P2.54mm_Vertical; DPN (none) -> WM4201-ND; DST (none) -> DigiKey; MFR (none) -> Molex; MPN (none) -> 22232031
- J8: renamed from J9; value Conn_01x03 -> 0022232031; DPN (none) -> WM4201-ND; DST (none) -> DigiKey; MFR (none) -> Molex; MPN (none) -> 22232031
- R24: renamed from R7; value 4.7 -> 4.7k; DPN (none) -> 311-4.70KHRCT-ND; DST (none) -> DigiKey; MFR (none) -> Yageo; MPN (none) -> RC0603FR-074K7L
- R32: footprint (none) -> Resistor_SMD:R_0603_1608Metric; DPN (none) -> 311-10.0KHRCT-ND; DST (none) -> DigiKey; MFR (none) -> Yageo; MPN (none) -> RC0603FR-0710KL
- R33: DPN (none) -> 311-15KGRCT-ND; DST (none) -> DigiKey; MFR (none) -> Yageo; MPN (none) -> RC0603JR-0715KL
- renumbered C21 to C16, C22 to C17, C23 to C18, C18 to C19, C17 to C20, C19 to C21, C20 to C22, D6 to D11, D3 to D12, D11 to D9, J5 to J6, J4 to J9, Q5 to Q2, Q4 to Q3, Q3 to Q4, Q2 to Q5, R28 to R21, R29 to R22, R27 to R23, R26 to R25, R22 to R26, R8 to R27, R30 to R28, R31 to R29, R23 to R30, R21 to R31, R25 to R34, R24 to R35, TP34 to TP12, TP33 to TP13, U4 to U3, U1 to U4
Connections:
- no-connect marks 24 -> 25

Commit message: Trace tweaks
Parts:
- added R36, R37: 100, Resistor_SMD:R_0603_1608Metric, symbol Device:R_Small_US
- SW1, SW2: DST (none) -> DigiKey
Connections:
- net at J7.1 (Pin_1): now also R37.1; no longer U3.36 (RXD0)
- net at J7.2 (Pin_2): now also R36.1; no longer U3.37 (TXD0)
- new net: R37.2, U3.36 (RXD0)
- new net: R36.2, U3.37 (TXD0)
Other:
- note added: "Transducer"
- note removed: "Debug LED"
- moved on the sheet: C16, J6, R21, R22
