File: pcb/rcs-controller.kicad_pcb (KiCad board)
At the start: 2 copper layers, 45.6 x 73 mm, 110 parts, among them J1 00222-32051, J10 0022-232021, J11 Conn_01x03, J2 0022-232021, J3 0022-232041, J4 Screw_Terminal_4_P3.50mm, J5 USB_C_Receptacle_USB2.0_14P, J6 Conn_01x03, J8 00222-32051, J9 Conn_01x03, Q1 SI7465DP-T1-E3, Q2 SI7465DP-T1-E3, Q3 SI7465DP-T1-E3, Q4 PMV45EN2, Q5 PMV45EN2, SW1 SW_Push, SW2 SW_Push, U1 LSM6DSOX, U2 MP26123DR-LF-Z, U3 TPS63070, U4 ESP32-S3-WROOM-1

Commit message: Finished BOM, changed holes to .3
Parts:
- moved R13 0.71 mm to (114.2, 133.2)
- moved C14 0.50 mm to (113.8, 131.0)
- renumbered C26 to C1, C11 to C10, C13 to C11, C14 to C12, C15 to C13, C16 to C14, C29 to C15, C21 to C16, C22 to C17, C23 to C18, C18 to C19, C1 to C2, C17 to C20, C19 to C21, C20 to C22, C2 to C3, C6 to C5, C7 to C6, C8 to C7, C9 to C8, C10 to C9, D13 to D1, D6 to D11, D3 to D12, D1 to D2, D2 to D3, D9 to D4, D4 to D5, D5 to D6, D11 to D9, J10 to J1, J11 to J10, J8 to J2, J1 to J3, J2 to J4, J3 to J5, J5 to J6, J6 to J7, J9 to J8, J4 to J9, Q5 to Q2, Q4 to Q3, Q3 to Q4, Q2 to Q5, R35 to R1, R36 to R2, R28 to R21, R29 to R22, R27 to R23, R7 to R24, R26 to R25, R22 to R26, R8 to R27, R30 to R28, R31 to R29, R1 to R3, R23 to R30, R21 to R31, R25 to R34, R24 to R35, R2 to R4, R3 to R5, R4 to R6, R5 to R7, R6 to R8, TP7 to TP10, TP9 to TP11, TP34 to TP12, TP33 to TP13, TP32 to TP6, TP30 to TP7, TP31 to TP8, TP6 to TP9, U2 to U1, U3 to U2, U4 to U3, U1 to U4
Routing:
- net +BATT: track 18.8 -> 18.0 mm
- net GND: vias 115 -> 113

Commit message: Updated version number and date
Routing:
- net GND: vias 113 -> 114
